File: ESP12Block.brd (EAGLE design)
At the start: 100 x 80 mm, 16 parts, among them U1 TPS5410DR

Commit message: minor changes
improved the 3.3V and GND paths
Parts:
- moved R4 0.91 mm to (26.1, 29.4)
- moved R2 0.64 mm to (27.3, 26.0)
- moved R3 0.64 mm to (25.2, 26.0)
- moved C4 0.50 mm to (22.9, 26.4)
Routing:
- net +3V3: track 37.8 -> 56.5 mm, vias 2 -> 1
- net GND: track 25.2 -> 7.83 mm, vias 4 -> 8
- net SENS: track 24.9 -> 23.3 mm
- net GPIO2: track 14.9 -> 13.6 mm
- net +12V: track 34.6 -> 33.4 mm
- net GPIO0: track 47.0 -> 46.4 mm
- net BOOT: track 7.61 -> 7.11 mm
- removed copper zone on layer 1, net +3V3
Other:
- board size 100 x 80 mm -> 32 x 32 mm
